Commit message: add additional configs,modify sensor config file, fix node spinning issue

File: gs_ros2_control_demos/urdf/test_diff_drive.xacro.urdf (robot description, URDF)
Before this commit: robot diff_drive, 4 links, 3 joints
Links:
- added link base_link
- added link camera_link, mass 0.01; collision box size=0.05 0.05 0.05; visual box size=0.05 0.05 0.05
- added link laser_link, mass 0.01; collision box size=0.05 0.05 0.05; visual box size=0.05 0.05 0.05
- added link lidar_link, mass 0.01; collision box size=0.05 0.05 0.05; visual box size=0.05 0.05 0.05
Joints:
- added joint camera_joint: type fixed, parent base_link, child camera_link, origin xyz=0 0 1.0 rpy=0 0 0
- added joint chassis_joint: type fixed, parent base_link, child chassis, origin xyz=0.8 0 0.5 rpy=0 0 0
- added joint laser_joint: type fixed, parent base_link, child laser_link, origin xyz=0 0.1 1.0 rpy=0 0 0
- added joint lidar_joint: type fixed, parent base_link, child lidar_link, origin xyz=0 -0.1 1.0 rpy=0 0 0

File: gs_ros2_control_demos/urdf/test_tricycle_drive.xacro.urdf (robot description, URDF)
Before this commit: robot tricycle_drive, 9 links, 8 joints
Joints:
- joint camera_joint: origin xyz=0 0 1.0 rpy=0 0 0 -> xyz=0.1 0 1.0 rpy=0 0 0
